Commit message: shin contacts

File: g1/21dof/g1_21dof.urdf (robot description, URDF)
Before this commit: robot g1_23dof_rev_1_0, 27 links, 26 joints
Links:
- link pelvis: geometry visual mesh filename=meshes/pelvis.STL
- link torso_link: geometry collision sphere radius=0.05; visual mesh filename=meshes/torso_link_23dof_rev_1_0.STL
